File: FANMONO.sch (KiCad schematic (older format))
At the start: 37 parts, among them P1 CONN_01X02, P2 CONN_01X02, P4 BDM, P5 CONN_01X03, P6 CONN_01X02, T1 TRANSFO, U1 78L05, U2 MC9S08SH8, U4 LM311N, U5 SSR_SHARP

Commit message: modificado componente ruteado
Parts:
- added C2: 0.1 uF, symbol C
- added P3: CONN_01X02, locales:PHOENIX_MSTBA2,54-G_2, symbol CONN_01X02
- added R2: 10k, Discret:R3, symbol R
- C1, C12, C8: footprint locales:C1 -> (none)
- D2, D4, D5: footprint Diodes_ThroughHole:Diode_DO-41_SOD81_Horizontal_RM10 -> (none)
- JP1, JP2, JP3: footprint Connect:PINHEAD1-2 -> (none)
- P5: footprint Connect:bornier3 -> (none)
- P6: footprint Connect:bornier2 -> (none)
- R10, R11, R3, R4, R7: footprint Discret:R3 -> (none)
- U2: symbol MC9S08SH8-RESCUE-FANMONO -> MC9S08SH8
- U4: footprint Housings_DIP:DIP-8_W7.62mm_LongPads -> (none)
- U5: footprint locales:SSR-SHARP -> (none)
Connections:
- net GM: now also C2.1, P3.2 (P2), R2.2
- net GND: now also C2.2, P3.1 (P1)
- net vreg: now also R2.1
Changed lines of the file:
@@
 EESchema Schematic File Version 2
-LIBS:FANMONO-rescue
 LIBS:power
 LIBS:device
@@
 Sheet 1 1
 Title "Protector de potencia"
-Date "30 nov 2015"
+Date "mar 17 nov 2015"
 Rev "1.0"
 Comp "Tecnitower"
@@
 vreg
 $Bitmap
-Pos 7988 7079
+Pos 7220 6750
 Scale 1,000000
 Data
@@
 $EndComp
 $Comp
-L MC9S08SH8-RESCUE-FANMONO U2
+L MC9S08SH8 U2
 U 1 1 5652FB51
 P 6325 4950
@@
 	1    0    0    -1
 $EndComp
+$Comp
+L CONN_01X02 P3
+U 1 1 5652FB87
+P 2030 4510
+F 0 "P3" H 2030 4660 50  0000 C CNN
+F 1 "CONN_01X02" V 2130 4510 50  0000 C CNN
+F 2 "locales:PHOENIX_MSTBA2,54-G_2" H 2030 4510 60  0001 C CNN
+F 3 "" H 2030 4510 60  0000 C CNN
+	1    2030 4510
+	-1   0    0    1
+$EndComp
+$Comp
+L R R2
+U 1 1 5652FB88
+P 2510 4220
+F 0 "R2" V 2590 4220 50  0000 C CNN
+F 1 "10k" V 2510 4220 50  0000 C CNN
+F 2 "Discret:R3" V 2440 4220 30  0001 C CNN
+F 3 "" H 2510 4220 30  0000 C CNN
+	1    2510 4220
+	1    0    0    -1
+$EndComp
 Text Label 875  615  0    60   ~ 0
 L
@@
 	1    0    0    -1
 $EndComp
+Text Label 2510 4020 2    60   ~ 0
+vreg
 Text Label 7775 5250 0    60   ~ 0
 AcOut
@@
 vreg
 $Comp
+L C C2
+U 1 1 56539B1C
+P 2510 4610
+F 0 "C2" H 2535 4710 50  0000 L CNN
+F 1 "0.1 uF" H 2535 4510 50  0000 L CNN
+F 2 "" H 2548 4460 30  0000 C CNN
+F 3 "" H 2510 4610 60  0000 C CNN
+	1    2510 4610
+	1    0    0    -1
+$EndComp
+$Comp
 L C C1
 U 1 1 5653A4FA
@@
 F 0 "C1" H 2530 5750 50  0000 L CNN
 F 1 "0.1 uF" H 2530 5550 50  0000 L CNN
-F 2 "locales:C1" H 2543 5500 30  0001 C CNN
+F 2 "" H 2543 5500 30  0000 C CNN
 F 3 "" H 2505 5650 60  0000 C CNN
 	1    2505 5650
 	1    0    0    -1
 $EndComp
+Text Label 2510 4460 2    60   ~ 0
+GM
 Text Label 2505 5500 2    60   ~ 0
 GP
@@
 F 0 "JP1" H 3390 4600 50  0000 C CNN
 F 1 "JUMPER" H 3390 4370 50  0000 C CNN
-F 2 "Connect:PINHEAD1-2" H 3390 4450 60  0001 C CNN
+F 2 "" H 3390 4450 60  0000 C CNN
 F 3 "" H 3390 4450 60  0000 C CNN
 	1    3390 4450
@@
 F 0 "D2" H 5805 5705 50  0000 C CNN
 F 1 "D" H 5915 5560 50  0000 C CNN
-F 2 "Diodes_ThroughHole:Diode_DO-41_SOD81_Horizontal_RM10" H 5915 5660 60  0001 C CNN
+F 2 "" H 5915 5660 60  0000 C CNN
 F 3 "" H 5915 5660 60  0000 C CNN
 	1    5915 5660
@@
 F 0 "JP3" H 5175 6290 50  0000 C CNN
 F 1 "JUMPER" H 5175 6060 50  0000 C CNN
-F 2 "Connect:PINHEAD1-2" H 5175 6140 60  0001 C CNN
+F 2 "" H 5175 6140 60  0000 C CNN
 F 3 "" H 5175 6140 60  0000 C CNN
 	1    5175 6140
@@
 F 0 "R4" V 5255 6620 50  0000 C CNN
 F 1 "R" V 5175 6620 50  0000 C CNN
-F 2 "Discret:R3" V 5105 6620 30  0001 C CNN
+F 2 "" V 5105 6620 30  0000 C CNN
 F 3 "" H 5175 6620 30  0000 C CNN
 	1    5175 6620
@@
 F 0 "JP2" H 3545 5725 50  0000 C CNN
 F 1 "JUMPER" H 3545 5495 50  0000 C CNN
-F 2 "Connect:PINHEAD1-2" H 3545 5575 60  0001 C CNN
+F 2 "" H 3545 5575 60  0000 C CNN
 F 3 "" H 3545 5575 60  0000 C CNN
 	1    3545 5575
@@
 F 0 "R3" V 3625 4975 50  0000 C CNN
 F 1 "R" V 3545 4975 50  0000 C CNN
-F 2 "Discret:R3" V 3475 4975 30  0001 C CNN
+F 2 "" V 3475 4975 30  0000 C CNN
 F 3 "" H 3545 4975 30  0000 C CNN
 	1    3545 4975
@@
 F 0 "U4" H 9490 3640 70  0000 C CNN
 F 1 "LM311N" H 9490 3540 70  0000 C CNN
-F 2 "Housings_DIP:DIP-8_W7.62mm_LongPads" H 9290 3340 60  0001 C CNN
+F 2 "" H 9290 3340 60  0000 C CNN
 F 3 "" H 9290 3340 60  0000 C CNN
 	1    9290 3340
@@
 F 0 "U5" H 9010 1520 60  0000 C CNN
 F 1 "SSR_SHARP" H 9010 1420 60  0000 C CNN
-F 2 "locales:SSR-SHARP" H 9010 1190 60  0001 C CNN
+F 2 "" H 9010 1190 60  0000 C CNN
 F 3 "" H 9010 1190 60  0000 C CNN
 	1    9010 1190
@@
 F 0 "D4" H 9510 1740 50  0000 C CNN
 F 1 "1N4148" H 9510 1540 50  0000 C CNN
-F 2 "Diodes_ThroughHole:Diode_DO-41_SOD81_Horizontal_RM10" H 9510 1640 60  0001 C CNN
+F 2 "" H 9510 1640 60  0000 C CNN
 F 3 "" H 9510 1640 60  0000 C CNN
 	1    9510 1640
@@
 F 0 "R11" V 9340 1790 50  0000 C CNN
 F 1 "220" V 9260 1790 50  0000 C CNN
-F 2 "Discret:R3" V 9190 1790 30  0001 C CNN
+F 2 "" V 9190 1790 30  0000 C CNN
 F 3 "" H 9260 1790 30  0000 C CNN
 	1    9260 1790
@@
 F 0 "C12" H 7850 1775 50  0000 L CNN
 F 1 "0.022 uF" H 7850 1575 50  0000 L CNN
-F 2 "locales:C1" H 7863 1525 30  0001 C CNN
+F 2 "" H 7863 1525 30  0000 C CNN
 F 3 "" H 7825 1675 60  0000 C CNN
 	1    7825 1675
@@
 F 0 "R7" V 7905 2010 50  0000 C CNN
 F 1 "47" V 7825 2010 50  0000 C CNN
-F 2 "Discret:R3" V 7755 2010 30  0001 C CNN
+F 2 "" V 7755 2010 30  0000 C CNN
 F 3 "" H 7825 2010 30  0000 C CNN
 	1    7825 2010
@@
 F 0 "P6" H 9765 2170 50  0000 C CNN
 F 1 "CONN_01X02" V 9865 2020 50  0000 C CNN
-F 2 "Connect:bornier2" H 9765 2020 60  0001 C CNN
+F 2 "" H 9765 2020 60  0000 C CNN
 F 3 "" H 9765 2020 60  0000 C CNN
 	1    9765 2020
@@
 Connection ~ 4440 5560
 Wire Wire Line
+	2510 4020 2510 4070
+Wire Wire Line
 	4875 4650 5175 4650
 Wire Wire Line
@@
 	2505 5060 2505 5110
 Wire Wire Line
+	2230 4460 2510 4460
+Wire Wire Line
+	2510 4460 2510 4370
+Wire Wire Line
 	2225 5800 2700 5800
+Wire Wire Line
+	2230 4560 2230 4815
 Wire Wire Line
 	2505 5410 2505 5500
@@
 F 0 "D5" H 3965 1565 40  0000 C CNN
 F 1 "DIODE" H 3965 1365 40  0000 C CNN
-F 2 "Diodes_ThroughHole:Diode_DO-41_SOD81_Horizontal_RM10" H 3965 1465 60  0001 C CNN
+F 2 "" H 3965 1465 60  0000 C CNN
 F 3 "" H 3965 1465 60  0000 C CNN
 	1    3965 1465
@@
 F 0 "C8" H 5585 6090 50  0000 L CNN
 F 1 "C" H 5585 5890 50  0000 L CNN
-F 2 "locales:C1" H 5598 5840 30  0001 C CNN
+F 2 "" H 5598 5840 30  0000 C CNN
 F 3 "" H 5560 5990 60  0000 C CNN
 	1    5560 5990
@@
 Connection ~ 5560 5760
 NoConn ~ 7775 5350
+Wire Wire Line
+	2230 4815 2510 4815
+Wire Wire Line
+	2510 4815 2510 4760
+$Comp
+L GND #PWR03
+U 1 1 5655064C
+P 2510 4815
+F 0 "#PWR03" H 2510 4565 50  0001 C CNN
+F 1 "GND" H 2510 4665 50  0000 C CNN
+F 2 "" H 2510 4815 60  0000 C CNN
+F 3 "" H 2510 4815 60  0000 C CNN
+	1    2510 4815
+	1    0    0    -1
+$EndComp
 Wire Wire Line
 	2505 5500 2225 5500
@@
 F 0 "P5" H 6360 5960 50  0000 C CNN
 F 1 "CONN_01X03" V 6460 5760 50  0000 C CNN
-F 2 "Connect:bornier3" H 6360 5760 60  0001 C CNN
+F 2 "" H 6360 5760 60  0000 C CNN
 F 3 "" H 6360 5760 60  0000 C CNN
 	1    6360 5760
@@
 F 0 "R10" V 10210 3620 50  0000 C CNN
 F 1 "10k" V 10130 3620 50  0000 C CNN
-F 2 "Discret:R3" V 10060 3620 30  0001 C CNN
+F 2 "" V 10060 3620 30  0000 C CNN
 F 3 "" H 10130 3620 30  0000 C CNN
 	1    10130 3620

Commit message: agregando valores de componentes
Parts:
- C8: value C -> 0,1 uF
- D2: value D -> 1N4007
- R3, R4: value R -> 10k
Changed lines of the file:
@@
 EESchema Schematic File Version 2
+LIBS:FANMONO-rescue
 LIBS:power
 LIBS:device
@@
 P 5915 5660
 F 0 "D2" H 5805 5705 50  0000 C CNN
-F 1 "D" H 5915 5560 50  0000 C CNN
+F 1 "1N4007" H 5915 5560 50  0000 C CNN
 F 2 "" H 5915 5660 60  0000 C CNN
 F 3 "" H 5915 5660 60  0000 C CNN
@@
 P 5175 6620
 F 0 "R4" V 5255 6620 50  0000 C CNN
-F 1 "R" V 5175 6620 50  0000 C CNN
+F 1 "10k" V 5175 6620 50  0000 C CNN
 F 2 "" V 5105 6620 30  0000 C CNN
 F 3 "" H 5175 6620 30  0000 C CNN
@@
 P 3545 4975
 F 0 "R3" V 3625 4975 50  0000 C CNN
-F 1 "R" V 3545 4975 50  0000 C CNN
+F 1 "10k" V 3545 4975 50  0000 C CNN
 F 2 "" V 3475 4975 30  0000 C CNN
 F 3 "" H 3545 4975 30  0000 C CNN
@@
 P 5560 5990
 F 0 "C8" H 5585 6090 50  0000 L CNN
-F 1 "C" H 5585 5890 50  0000 L CNN
+F 1 "0,1 uF" H 5585 5890 50  0000 L CNN
 F 2 "" H 5598 5840 30  0000 C CNN
 F 3 "" H 5560 5990 60  0000 C CNN
