File: FANMONO.sch (KiCad schematic (older format))
At the start: 40 parts, among them P1 CONN_01X02, P2 CONN_01X02, P3 CONN_01X02, P4 BDM, P5 CONN_01X03, P6 CONN_01X02, T1 TRANSFO, U1 78L05, U2 MC9S08SH8, U4 LM311N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

Commit message: realizando firmware
Parts:
- removed C2: 0.1 uF, symbol C
- removed JP1: JUMPER, symbol JUMPER
- removed P3: CONN_01X02, locales:PHOENIX_MSTBA2,54-G_2, symbol CONN_01X02
- removed R2: 10k, Discret:R3, symbol R
- added R12: 1 M, symbol R
- R5: value 10K -> 10k
Connections:
- net RESET is gone; now on net GP: C9.1, P4.4, R5.2, U2.1 (PTA5/IRQ/TCLK/RESET)
- net GND: now also C1.2, P2.1 (P1), R12.2
Changed lines of the file:
@@
 P 5890 3245
 F 0 "R5" V 5970 3245 50  0000 C CNN
-F 1 "10K" V 5890 3245 50  0000 C CNN
+F 1 "10k" V 5890 3245 50  0000 C CNN
 F 2 "Discret:R3" H 5890 3245 60  0001 C CNN
 F 3 "" H 5890 3245 60  0001 C CNN
@@
 	1    0    0    -1
 $EndComp
-$Comp
-L CONN_01X02 P3
-U 1 1 5652FB87
-P 2030 4510
-F 0 "P3" H 2030 4660 50  0000 C CNN
-F 1 "CONN_01X02" V 2130 4510 50  0000 C CNN
-F 2 "locales:PHOENIX_MSTBA2,54-G_2" H 2030 4510 60  0001 C CNN
-F 3 "" H 2030 4510 60  0000 C CNN
-	1    2030 4510
-	-1   0    0    1
-$EndComp
-$Comp
-L R R2
-U 1 1 5652FB88
-P 2510 4220
-F 0 "R2" V 2590 4220 50  0000 C CNN
-F 1 "10k" V 2510 4220 50  0000 C CNN
-F 2 "Discret:R3" V 2440 4220 30  0001 C CNN
-F 3 "" H 2510 4220 30  0000 C CNN
-	1    2510 4220
-	1    0    0    -1
-$EndComp
 Text Label 875  615  0    60   ~ 0
 L
@@
 	1    0    0    -1
 $EndComp
-Text Label 2510 4020 2    60   ~ 0
-vreg
 Text Label 7775 5250 0    60   ~ 0
 AcOut
@@
 vreg
 $Comp
-L C C2
-U 1 1 56539B1C
-P 2510 4610
-F 0 "C2" H 2535 4710 50  0000 L CNN
-F 1 "0.1 uF" H 2535 4510 50  0000 L CNN
-F 2 "" H 2548 4460 30  0000 C CNN
-F 3 "" H 2510 4610 60  0000 C CNN
-	1    2510 4610
-	1    0    0    -1
-$EndComp
-$Comp
 L C C1
 U 1 1 5653A4FA
@@
 	1    0    0    -1
 $EndComp
-Text Label 2510 4460 2    60   ~ 0
-GM
 Text Label 2505 5500 2    60   ~ 0
 GP
 Text Label 5000 4850 0    60   ~ 0
 GM
-$Comp
-L JUMPER JP1
-U 1 1 5653C692
-P 3390 4450
-F 0 "JP1" H 3390 4600 50  0000 C CNN
-F 1 "JUMPER" H 3390 4370 50  0000 C CNN
-F 2 "" H 3390 4450 60  0000 C CNN
-F 3 "" H 3390 4450 60  0000 C CNN
-	1    3390 4450
-	1    0    0    -1
-$EndComp
 $Comp
 L CONN_01X02 P1
@@
 Connection ~ 4440 5560
 Wire Wire Line
-	2510 4020 2510 4070
-Wire Wire Line
 	4875 4650 5175 4650
 Wire Wire Line
@@
 	2505 5060 2505 5110
 Wire Wire Line
-	2230 4460 2510 4460
-Wire Wire Line
-	2510 4460 2510 4370
-Wire Wire Line
-	2225 5800 2700 5800
-Wire Wire Line
-	2230 4560 2230 4815
-Wire Wire Line
 	2505 5410 2505 5500
-Wire Wire Line
-	2700 5800 2700 4450
 Connection ~ 2505 5500
 Wire Wire Line
-	2700 4450 3090 4450
-Wire Wire Line
-	3690 4450 3845 4450
-Wire Wire Line
-	3845 4450 3845 4395
-Wire Wire Line
-	3845 4395 4855 4395
+	2700 4395 4855 4395
 Wire Wire Line
 	4855 4395 4855 4450
@@
 NoConn ~ 7775 5350
 Wire Wire Line
-	2230 4815 2510 4815
-Wire Wire Line
-	2510 4815 2510 4760
-$Comp
-L GND #PWR03
-U 1 1 5655064C
-P 2510 4815
-F 0 "#PWR03" H 2510 4565 50  0001 C CNN
-F 1 "GND" H 2510 4665 50  0000 C CNN
-F 2 "" H 2510 4815 60  0000 C CNN
-F 3 "" H 2510 4815 60  0000 C CNN
-	1    2510 4815
-	1    0    0    -1
-$EndComp
-Wire Wire Line
-	2505 5500 2225 5500
+	2700 5500 2225 5500
 Wire Wire Line
 	5700 1465 5900 1465
@@
 	1    0    0    -1
 $EndComp
+$Comp
+L R R12
+U 1 1 5698FBE3
+P 8685 3490
+F 0 "R12" V 8765 3490 50  0000 C CNN
+F 1 "1 M" V 8685 3490 50  0000 C CNN
+F 2 "" V 8615 3490 30  0000 C CNN
+F 3 "" H 8685 3490 30  0000 C CNN
+	1    8685 3490
+	1    0    0    -1
+$EndComp
+$Comp
+L GND #PWR?
+U 1 1 5698FD10
+P 8685 3685
+F 0 "#PWR?" H 8685 3435 50  0001 C CNN
+F 1 "GND" H 8685 3535 50  0000 C CNN
+F 2 "" H 8685 3685 60  0000 C CNN
+F 3 "" H 8685 3685 60  0000 C CNN
+	1    8685 3685
+	1    0    0    -1
+$EndComp
+Wire Wire Line
+	8685 3685 8685 3640
+Wire Wire Line
+	2700 4395 2700 5500
+Wire Wire Line
+	2225 5800 2505 5800
+$Comp
+L GND #PWR?
+U 1 1 569D0A5A
+P 2505 5800
+F 0 "#PWR?" H 2505 5550 50  0001 C CNN
+F 1 "GND" H 2505 5650 50  0000 C CNN
+F 2 "" H 2505 5800 60  0000 C CNN
+F 3 "" H 2505 5800 60  0000 C CNN
+	1    2505 5800
+	1    0    0    -1
+$EndComp
