File: FANMONO.sch (KiCad schematic (older format))
At the start: 43 parts, among them P1 CONN_01X02, P2 CONN_01X03, P4 BDM, P5 CONN_01X03, P6 CONN_01X02, T1 TRANSFO, U1 78L05, U2 MC9S08SH8, U4 LM311N, U5 SSR_SHARP

Commit message: Terminado el ruteo de versión 2.0
Parts:
- removed JP1, JP2, JP3: JUMPER, Connect:PINHEAD1-2, symbol JUMPER
- added C11: 1 uF, symbol CAPAPOL
- added P3: JPS, Pin_Headers:Pin_Header_Angled_2x03, symbol CONN_02X03
- F1: footprint (none) -> Fuse_Holders_and_Fuses:Fuseholder5x20_horiz_SemiClosed_Casing10x25mm
- P4: footprint Pin_Headers:Pin_Header_Straight_2x03 -> Pin_Headers:Pin_Header_Angled_2x03
Connections:
- net GND: now also P3.2 (P2), P3.6 (P6)
- net N: now also F1.2; no longer P1.1 (P1)
- net vreg: now also C11.1
- net at C8.1, P5.2 (P2), U2.10 (PTC2/ADP10): now also P3.3 (P3)
- net MODE: now reaches R6.2, U2.11 (PTC1/TPM1CH1/ADP9)
- net MODE: now also C11.2, P3.5 (P5)
- net at R3.2, U2.6 (PTB6/SDA/XTAL): now also P3.1 (P1)
- net at F1.1: now also P1.1 (P1); no longer U5.2 (T2)
- net at P6.1 (P1): now also U5.2 (T2); no longer F1.2
- net T2: now reaches R4.1
- net T2: now also P3.4 (P4)
Other:
- moved on the sheet: C10, C6, C7, D1, D4, D5, F1, R9, T1, U1
