File: _saved_FANMONO.sch (KiCad schematic (older format))
At the start: 43 parts, among them P1 CONN_01X02, P2 CONN_01X03, P4 BDM, P5 CONN_01X03, P6 CONN_01X02, T1 TRANSFO, U1 78L05, U2 MC9S08SH8, U4 LM311N, U5 SSR_SHARP

Commit message: modificado el esquematico
Parts:
- F1: footprint (none) -> locales:portafusible
Changed lines of the file:
@@
 F 0 "F1" H 9040 2080 50  0000 C CNN
 F 1 "FUSE" H 9010 1920 50  0000 C CNN
-F 2 "" H 9110 1970 50  0001 C CNN
+F 2 "locales:portafusible" H 9110 1970 50  0001 C CNN
 F 3 "" H 9110 1970 50  0000 C CNN
 	1    9110 1970
